File: SUPERCLUSTER_mainboard/ballon.sch (EAGLE design)
At the start: 5 parts, among them J1 Qwiic Right Angle, X1 S4B-ZR

Commit message: PCB 0.2
Parts:
- added J2: MICRO-SD-PUSH-PUSH-EXT-PIN, SparkFun-Connectors:MICRO-SD-PUSH-PUSH-EXT-PIN
- added JP1, JP2, JP4: (no value), pinhead:PINHD-1X4
- added JP10: (no value), pinhead:PINHD-2X3
- added JP11: (no value), jumper:JP1Q
- added JP3: (no value), pinhead:PINHD-1X2
- added JP5: (no value), pinhead:PINHD-1X8
- added JP6, JP7, JP8, JP9: (no value), pinhead:PINHD-1X3
- added R2, R3, R4, R5, R6, R7, R8: 2k2, rcl:R-EU_0204/7
- added U1: RA-02_LORA, RA-02_LORA:RA-02_LORA
Connections:
- new net BAT+: JP3.1, R6.2, U$1.VSYS
- new net N$1: R7.2, R8.2
- new net N$3: JP11.2, R6.1, R7.1
- net +3V3: now also J2.VCC, JP1.2, JP10.1, JP10.3, JP10.5, JP2.2, JP4.1, JP5.3, R2.2, R3.2, R4.2, R5.2, U1.3.3V
- net ADC0: now also JP7.3
- net ADC1: now also JP7.2
- net ADC2: now also JP11.1, JP7.1
- net GND: now also J2.GND, JP1.1, JP10.2, JP10.4, JP10.6, JP2.1, JP3.2, JP4.4, JP5.4, R8.1, U1.GND
- net GPIO13: now also JP6.3
- net GPIO14: now also JP6.2
- net GPIO15: now also JP6.1
- net GPIO20: now also JP8.3
- net GPIO21: now also JP8.2
- net GPIO22: now also JP8.1
- net GPIO5: now also U1.NSS
- net GPIO6: now also U1.RESET
- net GPIO7: now also U1.DI00
- net GPIO8: now also J2.DAT3/!CS!
- net GPIO9: now also JP5.8
- net RX_0: now also JP4.3
- net SCL_0: now also JP1.4, JP2.4, R4.1
- net SCL_1: now also JP5.1, R5.1
- net SDA_0: now also JP1.3, JP2.3, R2.1
- net SDA_1: now also JP5.2, R3.1
- net SPI0_MISO: now also J2.DAT0/SDO, U1.MISO
- net SPI0_MOSI: now also J2.CMD/SDI, U1.MOSI
- net SPI0_SCK: now also J2.CLK/SCK, U1.SCK
- net SPI1_MISO: now also JP5.6, JP9.1
- net SPI1_MOSI: now also JP5.7, JP9.2
- net SPI1_SCK: now also JP5.5, JP9.3
- net TX_0: now also JP4.2
