File: SUPERCLUSTER_mainboard/ballon.sch (EAGLE design)
At the start: 25 parts, among them J1 Qwiic Right Angle, J2 MICRO-SD-PUSH-PUSH-EXT-PIN, U1 RA-02_LORA, X1 S4B-ZR

Commit message: PCB bugfix
Parts:
- JP11: device jumper:JP1Q -> pinhead:PINHD-1X2
Connections:
- net ADC2: now also JP11.2; no longer JP11.1
- net N$3: now also JP11.1; no longer JP11.2
Changed lines of the file:
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@@
 <part name="R8" library="rcl" library_urn="urn:adsk.eagle:library:334" deviceset="R-EU_" device="0204/7" package3d_urn="urn:adsk.eagle:package:23498/2" value="2k2"/>
 <part name="GND10" library="supply1" library_urn="urn:adsk.eagle:library:371" deviceset="GND" device=""/>
-<part name="JP11" library="jumper" library_urn="urn:adsk.eagle:library:252" deviceset="JP1Q" device="" package3d_urn="urn:adsk.eagle:package:15455/1"/>
 <part name="FRAME1" library="frames" library_urn="urn:adsk.eagle:library:229" deviceset="A3L-LOC" device=""/>
+<part name="JP11" library="pinhead" library_urn="urn:adsk.eagle:library:325" deviceset="PINHD-1X2" device="" package3d_urn="urn:adsk.eagle:package:22435/2"/>
 </parts>
 <sheets>
@@
 <attribute name="VALUE" x="129.54" y="180.34" size="1.778" layer="96"/>
 </instance>
-<instance part="JP11" gate="A" x="154.94" y="213.36" smashed="yes" rot="R90">
-<attribute name="NAME" x="160.02" y="210.82" size="1.778" layer="95" rot="R180"/>
-<attribute name="VALUE" x="160.02" y="217.805" size="1.778" layer="96" rot="R180"/>
-</instance>
 <instance part="FRAME1" gate="G$1" x="-63.5" y="-2.54" smashed="yes">
 <attribute name="DRAWING_NAME" x="280.67" y="12.7" size="2.54" layer="94"/>
 <attribute name="LAST_DATE_TIME" x="280.67" y="7.62" size="2.286" layer="94"/>
 <attribute name="SHEET" x="294.005" y="2.54" size="2.54" layer="94"/>
+</instance>
+<instance part="JP11" gate="G$1" x="157.48" y="223.52" smashed="yes" rot="R90">
+<attribute name="NAME" x="151.765" y="217.17" size="1.778" layer="95" rot="R90"/>
+<attribute name="VALUE" x="162.56" y="217.17" size="1.778" layer="96" rot="R90"/>
 </instance>
 </instances>
@@
 </segment>
 <segment>
-<pinref part="JP11" gate="A" pin="1"/>
-<wire x1="162.56" y1="213.36" x2="170.18" y2="213.36" width="0.1524" layer="91"/>
+<wire x1="157.48" y1="213.36" x2="170.18" y2="213.36" width="0.1524" layer="91"/>
 <label x="170.18" y="213.36" size="1.27" layer="95" xref="yes"/>
+<pinref part="JP11" gate="G$1" pin="2"/>
+<wire x1="157.48" y1="220.98" x2="157.48" y2="213.36" width="0.1524" layer="91"/>
 </segment>
 </net>
@@
 <wire x1="132.08" y1="210.82" x2="132.08" y2="213.36" width="0.1524" layer="91"/>
 <wire x1="132.08" y1="213.36" x2="132.08" y2="215.9" width="0.1524" layer="91"/>
-<wire x1="132.08" y1="213.36" x2="147.32" y2="213.36" width="0.1524" layer="91"/>
+<wire x1="132.08" y1="213.36" x2="154.94" y2="213.36" width="0.1524" layer="91"/>
 <junction x="132.08" y="213.36"/>
-<pinref part="JP11" gate="A" pin="2"/>
-</segment>
-</net>
+<pinref part="JP11" gate="G$1" pin="1"/>
+<wire x1="154.94" y1="213.36" x2="154.94" y2="220.98" width="0.1524" layer="91"/>
+</segment>
+</net>
