File: SUPERCLUSTER_mainboard/ballon.brd (EAGLE design)
At the start: 49.5 x 62.3 mm, 25 parts, among them J1 Qwiic Right Angle, J2 MICRO-SD-PUSH-PUSH-EXT-PIN, U1 RA-02_LORA, X1 S4B-ZR

Commit message: PCB bugfix
Parts:
- JP11: device jumper:JP1 -> pinhead:1X02
- moved JP11 1.27 mm to (41.9, 44.5), turned to 270 degrees
- flipped R8 to the top
Connections:
- net ADC2: now also JP11.2; no longer JP11.1
- net N$3: now also JP11.1; no longer JP11.2
Routing:
- net N$3: track 6.35 -> 5.08 mm
Changed lines of the file:
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@@
 </layers>
 <board>
+<fusionsync huburn="a.YnVzaW5lc3M6Z21haWwyNTY3ODk" projecturn="a.YnVzaW5lc3M6Z21haWwyNTY3ODkjRDIwMTkwNzI3MjA1NjkxMTgx" f3durn="urn:adsk.wipprod:dm.lineage:SSwDac2vTTKieOT2l55ejg" pcbguid="" lastpulledtime="" lastsyncedchangeguid="" latestrevisionid="a8b71ab4-e611-4249-8fe2-883fa49a639b" lastsyncedrevisionid="a8b71ab4-e611-4249-8fe2-883fa49a639b" lastboardhashguid="131e63d4-1610-8576-b97e-5781577898cd" lastpushedtime="2021-10-03T08:23:57Z" linktopcb3d="true"/>
 <plain>
 <wire x1="0" y1="0" x2="49.51" y2="0" width="0" layer="20"/>
@@
 <attribute name="VALUE" x="42.3926" y="50.4444" size="0.9906" layer="27" ratio="10" rot="R90"/>
 </element>
-<element name="R8" library="rcl" library_urn="urn:adsk.eagle:library:334" package="0204/7" package3d_urn="urn:adsk.eagle:package:23498/2" value="2k2" x="44.45" y="52.07" smashed="yes" rot="MR90">
-<attribute name="NAME" x="45.7454" y="49.53" size="0.9906" layer="26" ratio="10" rot="MR90"/>
-<attribute name="POPULARITY" value="79" x="44.45" y="52.07" size="1.778" layer="28" rot="MR90" display="off"/>
-<attribute name="SPICEPREFIX" value="R" x="44.45" y="52.07" size="1.778" layer="28" rot="MR90" display="off"/>
-<attribute name="VALUE" x="43.9674" y="50.4444" size="0.9906" layer="28" ratio="10" rot="MR90"/>
-</element>
-<element name="JP11" library="jumper" library_urn="urn:adsk.eagle:library:252" package="JP1" package3d_urn="urn:adsk.eagle:package:15455/1" value="" x="41.91" y="43.18" smashed="yes">
-<attribute name="NAME" x="40.259" y="40.64" size="1.27" layer="25" ratio="10" rot="R90"/>
-<attribute name="POPULARITY" value="15" x="41.91" y="43.18" size="1.778" layer="27" display="off"/>
-<attribute name="VALUE" x="44.831" y="40.64" size="1.27" layer="27" ratio="10" rot="R90"/>
+<element name="R8" library="rcl" library_urn="urn:adsk.eagle:library:334" package="0204/7" package3d_urn="urn:adsk.eagle:package:23498/2" value="2k2" x="44.45" y="52.07" smashed="yes" rot="R90">
+<attribute name="NAME" x="43.1546" y="49.53" size="0.9906" layer="25" ratio="10" rot="R90"/>
+<attribute name="POPULARITY" value="79" x="44.45" y="52.07" size="1.778" layer="27" rot="R90" display="off"/>
+<attribute name="SPICEPREFIX" value="R" x="44.45" y="52.07" size="1.778" layer="27" rot="R90" display="off"/>
+<attribute name="VALUE" x="44.9326" y="50.4444" size="0.9906" layer="27" ratio="10" rot="R90"/>
+</element>
+<element name="JP11" library="pinhead" library_urn="urn:adsk.eagle:library:325" package="1X02" package3d_urn="urn:adsk.eagle:package:22435/2" value="" x="41.91" y="44.45" smashed="yes" rot="R270">
+<attribute name="NAME" x="43.7388" y="47.0662" size="1.27" layer="25" ratio="10" rot="R270"/>
+<attribute name="POPULARITY" value="98" x="41.91" y="44.45" size="1.778" layer="27" rot="R270" display="off"/>
+<attribute name="VALUE" x="38.735" y="46.99" size="1.27" layer="27" rot="R270"/>
 </element>
 </elements>
@@
 <contactref element="U$1" pad="GP28_A2"/>
 <contactref element="JP7" pad="1"/>
-<contactref element="JP11" pad="1"/>
 <wire x1="33.655" y1="41.91" x2="36.83" y2="41.91" width="0.635" layer="1"/>
 <wire x1="44.45" y1="39.37" x2="45.72" y2="39.37" width="0.635" layer="1"/>
-<wire x1="44.45" y1="39.37" x2="41.91" y2="41.91" width="0.635" layer="1"/>
 <wire x1="36.83" y1="41.91" x2="39.37" y2="39.37" width="0.635" layer="1"/>
-<wire x1="39.37" y1="39.37" x2="45.72" y2="39.37" width="0.635" layer="1"/>
+<wire x1="39.37" y1="39.37" x2="41.91" y2="39.37" width="0.635" layer="1"/>
+<contactref element="JP11" pad="2"/>
+<wire x1="41.91" y1="39.37" x2="45.72" y2="39.37" width="0.635" layer="1"/>
+<wire x1="41.91" y1="43.18" x2="41.91" y2="39.37" width="0.635" layer="1"/>
 </signal>
 <signal name="GPIO20">
@@
 <contactref element="R7" pad="1"/>
 <contactref element="R6" pad="1"/>
-<contactref element="JP11" pad="2"/>
-<wire x1="41.91" y1="44.45" x2="41.91" y2="48.26" width="0.635" layer="1"/>
 <wire x1="41.91" y1="48.26" x2="39.37" y2="48.26" width="0.635" layer="1"/>
+<contactref element="JP11" pad="1"/>
+<wire x1="41.91" y1="45.72" x2="41.91" y2="48.26" width="0.635" layer="1"/>
 </signal>
 </signals>
@@
 </note>
 <note version="8.3" severity="warning">
+Since Version 8.3, EAGLE supports Fusion synchronisation.
+This feature will not be available in this version and saving
+the document will break the link to the Fusion PCB feature.
+</note>
+<note version="8.3" severity="warning">
